Commit message: Added third joint to the ROS firmware, though it is not manipulable with the DiffDrive controller

File: arm-ros-firmware/description/ros2_control/diffbot.ros2_control.xacro (robot description, xacro)
@@ -16,10 +16,15 @@
         </hardware>
       </xacro:if>
-      <joint name="${prefix}left_wheel_joint">
+      <joint name="${prefix}base_yaw_joint">
         <command_interface name="velocity"/>
         <state_interface name="position"/>
         <state_interface name="velocity"/>
       </joint>
-      <joint name="${prefix}right_wheel_joint">
+      <joint name="${prefix}base_pitch_joint">
+        <command_interface name="velocity"/>
+        <state_interface name="position"/>
+        <state_interface name="velocity"/>
+      </joint>
+      <joint name="${prefix}elbow_0_joint">
         <command_interface name="velocity"/>
         <state_interface name="position"/>
