Commit message: Finished renaming

File: description/ros2_control/prairie_pioneer.ros2_control.xacro (robot description, xacro)
@@ -1,5 +1,5 @@
 <?xml version="1.0"?>
 <robot xmlns:xacro="http://www.ros.org/wiki/xacro">
-  <xacro:macro name="diffbot_ros2_control" params="name prefix use_mock_hardware">
+  <xacro:macro name="prairie_pioneer_ros2_control" params="name prefix use_mock_hardware">
     <ros2_control name="${name}" type="system">
       <xacro:unless value="${use_mock_hardware}">

File: description/urdf/prairie_pioneer.urdf.xacro (robot description, xacro)
@@ -4,11 +4,11 @@
   <xacro:arg name="prefix" default="" />
   <xacro:arg name="use_mock_hardware" default="false" />
-  <xacro:include filename="$(find umrt-arm-ros-firmware)/ros2_control_demo_description/diffbot/urdf/diffbot_description.urdf.xacro" />
+  <xacro:include filename="$(find umrt-arm-ros-firmware)/ros2_control_demo_description/prairie_pioneer/urdf/prairie_pioneer_description.urdf.xacro" />
   <!-- Import Rviz colors -->
-  <xacro:include filename="$(find umrt-arm-ros-firmware)/ros2_control_demo_description/diffbot/urdf/diffbot.materials.xacro" />
-  <!-- Import diffbot ros2_control description -->
+  <xacro:include filename="$(find umrt-arm-ros-firmware)/ros2_control_demo_description/prairie_pioneer/urdf/prairie_pioneer.materials.xacro" />
+  <!-- Import prairie_pioneer ros2_control description -->
   <xacro:include filename="$(find umrt-arm-ros-firmware)/ros2_control/prairie_pioneer.ros2_control.xacro" />
-  <xacro:diffbot prefix="$(arg prefix)" />
-  <xacro:diffbot_ros2_control
-    name="DiffBot" prefix="$(arg prefix)" use_mock_hardware="$(arg use_mock_hardware)"/>
+  <xacro:prairie_pioneer prefix="$(arg prefix)" />
+  <xacro:prairie_pioneer_ros2_control
+    name="PrairiePioneer" prefix="$(arg prefix)" use_mock_hardware="$(arg use_mock_hardware)"/>
 </robot>

File: hardware/include/ros2_control_demo_description/prairie_pioneer/urdf/prairie_pioneer_description.urdf.xacro (robot description, xacro)
@@ -1,5 +1,5 @@
 <?xml version="1.0"?>
 <robot xmlns:xacro="http://www.ros.org/wiki/xacro">
-  <xacro:macro name="diffbot" params="prefix">
+  <xacro:macro name="prairie_pioneer" params="prefix">
   <!-- Constants for robot dimensions -->
   <xacro:property name="PI" value="3.1415926535897931"/>
