Commit message: Converted rviz stuff from diffbot to rrbot for experimentation

File: description/urdf/project_perry.urdf.xacro (robot description, xacro)
@@ -9,5 +9,9 @@
   <!-- Import project_perry ros2_control description -->
   <xacro:include filename="$(find umrt-arm-ros-firmware)/ros2_control/project_perry.ros2_control.xacro" />
-  <xacro:project_perry prefix="$(arg prefix)" />
+  <!-- Used for fixing robot -->
+  <link name="world"/>
+  <xacro:project_perry parent="world" prefix="$(arg prefix)">
+          <origin xyz="0 0 0" rpy="0 0 0" />
+  </xacro:project_perry>
   <xacro:project_perry_ros2_control
     name="ProjectPerry" prefix="$(arg prefix)" use_mock_hardware="$(arg use_mock_hardware)"/>

File: hardware/include/ros2_control_demo_description/project_perry/urdf/project_perry.materials.xacro (robot description, xacro)
@@ -20,4 +20,7 @@
     <color rgba="${255/255} ${108/255} ${10/255} 1.0"/>
   </material>
+  <material name="yellow">
+    <color rgba="${255/255} ${10/255} ${255/255} 1.0"/>
+  </material>
   <material name="brown">
     <color rgba="${222/255} ${207/255} ${195/255} 1.0"/>

File: hardware/include/ros2_control_demo_description/project_perry/urdf/project_perry_description.urdf.xacro (robot description, xacro)
@@ -1,163 +1,146 @@
 <?xml version="1.0"?>
 <robot xmlns:xacro="http://www.ros.org/wiki/xacro">
-  <xacro:macro name="project_perry" params="prefix">
-  <!-- Constants for robot dimensions -->
-  <xacro:property name="PI" value="3.1415926535897931"/>
-  <xacro:property name="base_mass" value="0.3" /> <!-- arbitrary value for base mass -->
-  <xacro:property name="base_width" value="0.1" />
-  <xacro:property name="base_length" value="0.1" />
-  <xacro:property name="base_height" value="0.05" />
-  <xacro:property name="wheel_mass" value="0.3" /> <!-- arbitrary value for wheel mass -->
-  <xacro:property name="wheel_len" value="0.020" />
-  <xacro:property name="wheel_radius" value="0.015" />
-  <xacro:property name="caster_wheel_mass" value="0.1" /> <!-- arbitrary value for caster wheel mass -->
-  <xacro:property name="caster_wheel_radius" value="0.015" />
-  <xacro:property name="z_offset" value="-${base_height/2}" /> <!-- Space btw top of beam and the each joint -->
-  <!-- Base Link -->
-  <link name="${prefix}base_link">
-    <collision>
-      <origin xyz="0 0 0" rpy="0 0 0"/>
-      <geometry>
-        <box size="${base_width} ${base_length} ${base_height}"/>
-      </geometry>
-    </collision>
-    <visual>
-      <origin xyz="0 0 ${base_height/2}" rpy="0 0 0"/>
-      <geometry>
-        <box size="${base_width} ${base_length} ${base_height}"/>
-      </geometry>
-      <material name="orange"/>
-    </visual>
-    <inertial>
-      <origin xyz="0 0 0" rpy="0 0 0"/>
-      <mass value="${base_mass}"/>
-      <inertia
-        ixx="${base_mass / 12.0 * (base_length*base_length + base_height*base_height)}" ixy="0.0" ixz="0.0"
-        iyy="${base_mass / 12.0 * (base_height*base_height + base_width*base_width)}" iyz="0.0"
-        izz="${base_mass / 12.0 * (base_width*base_width + base_length*base_length)}"/>
-      </inertial>
-    </link>
-    <joint name="${prefix}left_wheel_joint" type="continuous">
-      <parent link="${prefix}base_link"/>
-      <child link="${prefix}left_wheel"/>
-      <origin xyz="0 -${base_width/2} ${z_offset}" rpy="0 0 0"/>
-      <axis xyz="0 1 0"/>
-      <dynamics damping="0.2"/>
-      <limit effort="100" velocity="1.0"/>
-    </joint>
-    <!-- left wheel Link -->
-    <link name="${prefix}left_wheel">
-      <collision>
-        <origin xyz="0 0 0" rpy="${PI/2} 0 0"/>
-        <geometry>
-          <cylinder length="${wheel_len}" radius="${wheel_radius}"/>
-        </geometry>
-      </collision>
-      <visual>
-        <origin xyz="0 0 0" rpy="${PI/2} 0 0"/>
-        <geometry>
-          <cylinder length="${wheel_len}" radius="${wheel_radius}"/>
-        </geometry>
-        <material name="black"/>
-      </visual>
-      <inertial>
-        <origin xyz="0 0 0" rpy="${PI/2} 0 0"/>
-        <mass value="${wheel_mass}"/>
-        <inertia
-          ixx="${wheel_mass / 12.0 * (3*wheel_radius*wheel_radius + wheel_len*wheel_len)}" ixy="0.0" ixz="0.0"
-          iyy="${wheel_mass / 12.0 * (3*wheel_radius*wheel_radius + wheel_len*wheel_len)}" iyz="0.0"
-          izz="${wheel_mass / 2.0 * wheel_radius*wheel_radius}"/>
-        </inertial>
-      </link>
-    <joint name="${prefix}right_wheel_joint" type="continuous">
-      <parent link="${prefix}base_link"/>
-      <child link="${prefix}right_wheel"/>
-      <origin xyz="0 ${base_width/2} ${z_offset}" rpy="0 0 0"/>
-      <axis xyz="0 1 0"/>
-      <dynamics damping="0.2"/>
-      <limit effort="100" velocity="1.0"/>
-    </joint>
-    <!-- right wheel Link -->
-    <link name="${prefix}right_wheel">
-      <collision>
-        <origin xyz="0 0 0" rpy="${PI/2} 0 0"/>
-        <geometry>
-          <cylinder length="${wheel_len}" radius="${wheel_radius}"/>
-        </geometry>
-      </collision>
-      <visual>
-        <origin xyz="0 0 0" rpy="${PI/2} 0 0"/>
-        <geometry>
-          <cylinder length="${wheel_len}" radius="${wheel_radius}"/>
-        </geometry>
-        <material name="black"/>
-      </visual>
-      <inertial>
-        <origin xyz="0 0 0" rpy="${PI/2} 0 0"/>
-        <mass value="${wheel_mass}"/>
-        <inertia
-          ixx="${wheel_mass / 12.0 * (3*wheel_radius*wheel_radius + wheel_len*wheel_len)}" ixy="0.0" ixz="0.0"
-          iyy="${wheel_mass / 12.0 * (3*wheel_radius*wheel_radius + wheel_len*wheel_len)}" iyz="0.0"
-          izz="${wheel_mass / 2.0 * wheel_radius*wheel_radius}"/>
-        </inertial>
-      </link>
-    <joint name="${prefix}caster_frontal_wheel_joint" type="fixed">
-      <parent link="${prefix}base_link"/>
-      <child link="${prefix}caster_frontal_wheel"/>
-      <origin xyz="${base_width/2 - caster_wheel_radius} 0 ${z_offset}" rpy="0 0 0"/>
-    </joint>
-    <!-- caster frontal wheel Link -->
-    <link name="${prefix}caster_frontal_wheel">
-      <collision>
-        <origin xyz="0 0 0" rpy="0 0 0"/>
-        <geometry>
-          <sphere radius="${caster_wheel_radius}"/>
-        </geometry>
-      </collision>
-      <visual>
-        <origin xyz="0 0 0" rpy="0 0 0"/>
-        <geometry>
-          <sphere radius="${caster_wheel_radius}"/>
-        </geometry>
-        <material name="white"/>
-      </visual>
-      <inertial>
-        <origin xyz="0 0 0" rpy="0 0 0"/>
-        <mass value="${caster_wheel_mass}"/>
-        <inertia
-          ixx="${caster_wheel_mass * 0.4 * (caster_wheel_radius * caster_wheel_radius)}" ixy="0.0" ixz="0.0"
-          iyy="${caster_wheel_mass * 0.4 * (caster_wheel_radius * caster_wheel_radius)}" iyz="0.0"
-          izz="${caster_wheel_mass * 0.4 * (caster_wheel_radius * caster_wheel_radius)}"/>
-        </inertial>
-      </link>
-    <joint name="${prefix}caster_rear_wheel_joint" type="fixed">
-      <parent link="${prefix}base_link"/>
-      <child link="${prefix}caster_rear_wheel"/>
-      <origin xyz="${-base_width/2 + caster_wheel_radius} 0 ${z_offset}" rpy="0 0 0"/>
-    </joint>
-    <!-- caster rear wheel Link -->
-    <link name="${prefix}caster_rear_wheel">
-      <collision>
-        <origin xyz="0 0 0" rpy="0 0 0"/>
-        <geometry>
-          <sphere radius="${caster_wheel_radius}"/>
-        </geometry>
-      </collision>
-      <visual>
-        <origin xyz="0 0 0" rpy="0 0 0"/>
-        <geometry>
-          <sphere radius="${caster_wheel_radius}"/>
-        </geometry>
-        <material name="white"/>
-      </visual>
-      <inertial>
-        <origin xyz="0 0 0" rpy="0 0 0"/>
-        <mass value="${caster_wheel_mass}"/>
-        <inertia
-          ixx="${caster_wheel_mass * 0.4 * (caster_wheel_radius * caster_wheel_radius)}" ixy="0.0" ixz="0.0"
-          iyy="${caster_wheel_mass * 0.4 * (caster_wheel_radius * caster_wheel_radius)}" iyz="0.0"
-          izz="${caster_wheel_mass * 0.4 * (caster_wheel_radius * caster_wheel_radius)}"/>
-        </inertial>
-      </link>
-  </xacro:macro>
+    <xacro:macro name="project_perry" params="parent prefix *origin">
+        <!-- Constants for robot dimensions -->
+        <xacro:property name="mass" value="1"/> <!-- arbitrary value for mass -->
+        <xacro:property name="width" value="0.1"/> <!-- Square dimensions (widthxwidth) of beams -->
+        <xacro:property name="height1" value="2"/> <!-- Link 1 -->
+        <xacro:property name="height2" value="1"/> <!-- Link 2 -->
+        <xacro:property name="height3" value="1"/> <!-- Link 3 -->
+        <xacro:property name="axel_offset" value="0.05"/> <!-- Space btw top of beam and the each joint -->
+        <joint name="${prefix}base_joint" type="fixed">
+            <xacro:insert_block name="origin"/>
+            <parent link="${parent}"/>
+            <child link="${prefix}base_link"/>
+        </joint>
+        <!-- Base Link -->
+        <link name="${prefix}base_link">
+            <collision>
+                <origin xyz="0 0 ${height1/2}" rpy="0 0 0"/>
+                <geometry>
+                    <box size="${width} ${width} ${height1}"/>
+                </geometry>
+            </collision>
+            <visual>
+                <origin xyz="0 0 ${height1/2}" rpy="0 0 0"/>
+                <geometry>
+                    <box size="${width} ${width} ${height1}"/>
+                </geometry>
+                <material name="orange"/>
+            </visual>
+            <inertial>
+                <origin xyz="0 0 ${height1/2}" rpy="0 0 0"/>
+                <mass value="${mass}"/>
+                <inertia
+                        ixx="${mass / 12.0 * (width*width + height1*height1)}" ixy="0.0" ixz="0.0"
+                        iyy="${mass / 12.0 * (height1*height1 + width*width)}" iyz="0.0"
+                        izz="${mass / 12.0 * (width*width + width*width)}"/>
+            </inertial>
+        </link>
+        <joint name="${prefix}base_yaw_joint" type="continuous">
+            <parent link="${prefix}base_link"/>
+            <child link="${prefix}shoulder_link"/>
+            <origin xyz="0 ${width} ${height1 - axel_offset}" rpy="0 0 0"/>
+            <axis xyz="0 1 0"/>
+            <dynamics damping="0.7"/>
+            <limit effort="100" velocity="1.0"/>
+        </joint>
+        <!-- Middle Link -->
+        <link name="${prefix}shoulder_link">
+            <collision>
+                <origin xyz="0 0 ${height2/2 - axel_offset}" rpy="0 0 0"/>
+                <geometry>
+                    <box size="${width} ${width} ${height2}"/>
+                </geometry>
+            </collision>
+            <visual>
+                <origin xyz="0 0 ${height2/2 - axel_offset}" rpy="0 0 0"/>
+                <geometry>
+                    <box size="${width} ${width} ${height2}"/>
+                </geometry>
+                <material name="yellow"/>
+            </visual>
+            <inertial>
+                <origin xyz="0 0 ${height2/2 - axel_offset}" rpy="0 0 0"/>
+                <mass value="${mass}"/>
+                <inertia
+                        ixx="${mass / 12.0 * (width*width + height2*height2)}" ixy="0.0" ixz="0.0"
+                        iyy="${mass / 12.0 * (height2*height2 + width*width)}" iyz="0.0"
+                        izz="${mass / 12.0 * (width*width + width*width)}"/>
+            </inertial>
+        </link>
+        <joint name="${prefix}base_pitch_joint" type="continuous">
+            <parent link="${prefix}shoulder_link"/>
+            <child link="${prefix}humerus_link"/>
+            <origin xyz="0 ${width} ${height2 - axel_offset*2}" rpy="0 0 0"/>
+            <axis xyz="0 1 0"/>
+            <dynamics damping="0.7"/>
+            <limit effort="100" velocity="1.0"/>
+        </joint>
+        <!-- Top Link -->
+        <link name="${prefix}humerus_link">
+            <collision>
+                <origin xyz="0 0 ${height3/2 - axel_offset}" rpy="0 0 0"/>
+                <geometry>
+                    <box size="${width} ${width} ${height3}"/>
+                </geometry>
+            </collision>
+            <visual>
+                <origin xyz="0 0 ${height3/2 - axel_offset}" rpy="0 0 0"/>
+                <geometry>
+                    <box size="${width} ${width} ${height3}"/>
+                </geometry>
+                <material name="orange"/>
+            </visual>
+            <inertial>
+                <origin xyz="0 0 ${height3/2 - axel_offset}" rpy="0 0 0"/>
+                <mass value="${mass}"/>
+                <inertia
+                        ixx="${mass / 12.0 * (width*width + height3*height3)}" ixy="0.0" ixz="0.0"
+                        iyy="${mass / 12.0 * (height3*height3 + width*width)}" iyz="0.0"
+                        izz="${mass / 12.0 * (width*width + width*width)}"/>
+            </inertial>
+        </link>
+        <joint name="${prefix}elbow_0_joint" type="continuous">
+            <origin xyz="0 0 1" rpy="0 0 0"/>
+            <parent link="${prefix}humerus_link"/>
+            <child link="${prefix}gripper_link"/>
+            <origin xyz="0 ${width} ${height3 - axel_offset*3}" rpy="0 0 0"/>
+            <axis xyz="0 1 0"/>
+            <dynamics damping="0.7"/>
+            <limit effort="100" velocity="1.0"/>
+        </joint>
+        <!-- Gripper Link -->
+        <link name="${prefix}gripper_link">
+            <collision>
+                <origin xyz="0 0 ${height3/2 - axel_offset}" rpy="0 0 0"/>
+                <geometry>
+                    <box size="${width} ${width} ${height3}"/>
+                </geometry>
+            </collision>
+            <visual>
+                <origin xyz="0 0 ${height3/2 - axel_offset}" rpy="0 0 0"/>
+                <geometry>
+                    <box size="${width} ${width} ${height3}"/>
+                </geometry>
+                <material name="orange"/>
+            </visual>
+            <inertial>
+                <origin xyz="0 0 ${height3/2 - axel_offset}" rpy="0 0 0"/>
+                <mass value="${mass}"/>
+                <inertia
+                        ixx="${mass / 12.0 * (width*width + height3*height3)}" ixy="0.0" ixz="0.0"
+                        iyy="${mass / 12.0 * (height3*height3 + width*width)}" iyz="0.0"
+                        izz="${mass / 12.0 * (width*width + width*width)}"/>
+            </inertial>
+        </link>
+        <joint name="${prefix}gripper" type="fixed">
+            <origin xyz="0 0 1" rpy="0 0 0"/>
+            <parent link="${prefix}gripper_link"/>
+            <child link="${prefix}tool_link"/>
+        </joint>
+        <!-- Tool Link -->
+        <link name="${prefix}tool_link">
+        </link>
+    </xacro:macro>
 </robot>
