Commit message: Made model look more like prairie pioneer

File: hardware/include/ros2_control_demo_description/project_perry/urdf/project_perry_description.urdf.xacro (robot description, xacro)
@@ -4,4 +4,8 @@
         <!-- Constants for robot dimensions -->
         <xacro:property name="mass" value="1"/> <!-- arbitrary value for mass -->
+        <xacro:property name="base_width" value="1"/>
+        <xacro:property name="base_height" value="0.6"/>
+        <xacro:property name="platter_radius" value="0.75"/>
+        <xacro:property name="platter_height" value="0.1"/>
         <xacro:property name="width" value="0.1"/> <!-- Square dimensions (widthxwidth) of beams -->
         <xacro:property name="height1" value="2"/> <!-- Link 1 -->
@@ -17,23 +21,23 @@
         <link name="${prefix}base_link">
             <collision>
-                <origin xyz="0 0 ${height1/2}" rpy="0 0 0"/>
+                <origin xyz="0 0 ${base_height/2}" rpy="0 0 0"/>
                 <geometry>
-                    <box size="${width} ${width} ${height1}"/>
+                    <box size="${base_width} ${base_width} ${base_height}"/>
                 </geometry>
             </collision>
             <visual>
-                <origin xyz="0 0 ${height1/2}" rpy="0 0 0"/>
+                <origin xyz="0 0 ${base_height/2}" rpy="0 0 0"/>
                 <geometry>
-                    <box size="${width} ${width} ${height1}"/>
+                    <box size="${base_width} ${base_width} ${base_height}"/>
                 </geometry>
                 <material name="orange"/>
             </visual>
             <inertial>
-                <origin xyz="0 0 ${height1/2}" rpy="0 0 0"/>
+                <origin xyz="0 0 ${base_height/2}" rpy="0 0 0"/>
                 <mass value="${mass}"/>
                 <inertia
-                        ixx="${mass / 12.0 * (width*width + height1*height1)}" ixy="0.0" ixz="0.0"
-                        iyy="${mass / 12.0 * (height1*height1 + width*width)}" iyz="0.0"
-                        izz="${mass / 12.0 * (width*width + width*width)}"/>
+                        ixx="${mass / 12.0 * (base_width*base_width + base_height*base_height)}" ixy="0.0" ixz="0.0"
+                        iyy="${mass / 12.0 * (base_height*base_height + base_width*base_width)}" iyz="0.0"
+                        izz="${mass / 12.0 * (base_width*base_width + base_width*base_width)}"/>
             </inertial>
         </link>
@@ -41,6 +45,6 @@
             <parent link="${prefix}base_link"/>
             <child link="${prefix}shoulder_link"/>
-            <origin xyz="0 ${width} ${height1 - axel_offset}" rpy="0 0 0"/>
-            <axis xyz="0 1 0"/>
+            <origin xyz="0 0 ${base_height - axel_offset}" rpy="0 0 0"/>
+            <axis xyz="0 0 1"/>
             <dynamics damping="0.7"/>
             <limit effort="100" velocity="1.0"/>
@@ -49,32 +53,32 @@
         <link name="${prefix}shoulder_link">
             <collision>
-                <origin xyz="0 0 ${height2/2 - axel_offset}" rpy="0 0 0"/>
+                <origin xyz="0 0 ${platter_height/2 + axel_offset}" rpy="0 0 0"/>
                 <geometry>
-                    <box size="${width} ${width} ${height2}"/>
+                    <cylinder radius="${platter_radius}" length="${platter_height}"/>
                 </geometry>
             </collision>
             <visual>
-                <origin xyz="0 0 ${height2/2 - axel_offset}" rpy="0 0 0"/>
+                <origin xyz="0 0 ${platter_height/2 + axel_offset}" rpy="0 0 0"/>
                 <geometry>
-                    <box size="${width} ${width} ${height2}"/>
+                    <cylinder radius="${platter_radius}" length="${platter_height}"/>
                 </geometry>
                 <material name="yellow"/>
             </visual>
             <inertial>
-                <origin xyz="0 0 ${height2/2 - axel_offset}" rpy="0 0 0"/>
+                <origin xyz="0 0 ${platter_height/2 - axel_offset}" rpy="0 0 0"/>
                 <mass value="${mass}"/>
                 <inertia
-                        ixx="${mass / 12.0 * (width*width + height2*height2)}" ixy="0.0" ixz="0.0"
-                        iyy="${mass / 12.0 * (height2*height2 + width*width)}" iyz="0.0"
-                        izz="${mass / 12.0 * (width*width + width*width)}"/>
+                        ixx="${mass / 12.0 * (3*platter_radius*platter_radius + platter_height*platter_height)}" ixy="0.0" ixz="0.0"
+                        iyy="${mass / 12.0 * (3*platter_radius*platter_radius + platter_height*platter_height)}" iyz="0.0"
+                        izz="${mass / 2.0 * platter_radius*platter_radius}"/>
             </inertial>
         </link>
-        <joint name="${prefix}base_pitch_joint" type="continuous">
+        <joint name="${prefix}base_pitch_joint" type="revolute">
             <parent link="${prefix}shoulder_link"/>
             <child link="${prefix}humerus_link"/>
-            <origin xyz="0 ${width} ${height2 - axel_offset*2}" rpy="0 0 0"/>
+            <origin xyz="0 0 ${platter_height + axel_offset*2}" rpy="0 0 0"/>
             <axis xyz="0 1 0"/>
             <dynamics damping="0.7"/>
-            <limit effort="100" velocity="1.0"/>
+            <limit lower="${-pi/2.0}" upper="${pi/2.0}" effort="100" velocity="1.0"/>
         </joint>
         <!-- Top Link -->
@@ -102,12 +106,11 @@
             </inertial>
         </link>
-        <joint name="${prefix}elbow_0_joint" type="continuous">
-            <origin xyz="0 0 1" rpy="0 0 0"/>
+        <joint name="${prefix}elbow_0_joint" type="revolute">
             <parent link="${prefix}humerus_link"/>
             <child link="${prefix}gripper_link"/>
-            <origin xyz="0 ${width} ${height3 - axel_offset*3}" rpy="0 0 0"/>
+            <origin xyz="0 0 ${height3}" rpy="0 0 0"/>
             <axis xyz="0 1 0"/>
             <dynamics damping="0.7"/>
-            <limit effort="100" velocity="1.0"/>
+            <limit lower="${-3*pi/4.0}" upper="${3*pi/4.0}" effort="100" velocity="1.0"/>
         </joint>
         <!-- Gripper Link -->

Commit message: Added gripper

File: hardware/include/ros2_control_demo_description/project_perry/urdf/project_perry_description.urdf.xacro (robot description, xacro)
@@ -12,4 +12,9 @@
         <xacro:property name="height2" value="1"/> <!-- Link 2 -->
         <xacro:property name="height3" value="1"/> <!-- Link 3 -->
+        <xacro:property name="gripper_width" value="0.4"/>
+        <xacro:property name="gripper_breadth" value="0.1"/>
+        <xacro:property name="gripper_thickness" value="0.05"/>
+        <xacro:property name="finger_length" value="0.2"/>
+        <xacro:property name="finger_thickness" value="0.05"/>
         <xacro:property name="axel_offset" value="0.05"/> <!-- Space btw top of beam and the each joint -->
         <joint name="${prefix}base_joint" type="fixed">
@@ -69,6 +74,8 @@
                 <mass value="${mass}"/>
                 <inertia
-                        ixx="${mass / 12.0 * (3*platter_radius*platter_radius + platter_height*platter_height)}" ixy="0.0" ixz="0.0"
-                        iyy="${mass / 12.0 * (3*platter_radius*platter_radius + platter_height*platter_height)}" iyz="0.0"
+                        ixx="${mass / 12.0 * (3*platter_radius*platter_radius + platter_height*platter_height)}"
+                        ixy="0.0" ixz="0.0"
+                        iyy="${mass / 12.0 * (3*platter_radius*platter_radius + platter_height*platter_height)}"
+                        iyz="0.0"
                         izz="${mass / 2.0 * platter_radius*platter_radius}"/>
             </inertial>
@@ -108,5 +115,5 @@
         <joint name="${prefix}elbow_0_joint" type="revolute">
             <parent link="${prefix}humerus_link"/>
-            <child link="${prefix}gripper_link"/>
+            <child link="${prefix}wrist_link"/>
             <origin xyz="0 0 ${height3}" rpy="0 0 0"/>
             <axis xyz="0 1 0"/>
@@ -114,6 +121,6 @@
             <limit lower="${-3*pi/4.0}" upper="${3*pi/4.0}" effort="100" velocity="1.0"/>
         </joint>
-        <!-- Gripper Link -->
-        <link name="${prefix}gripper_link">
+        <!-- Wrist Link -->
+        <link name="${prefix}wrist_link">
             <collision>
                 <origin xyz="0 0 ${height3/2 - axel_offset}" rpy="0 0 0"/>
@@ -138,11 +145,96 @@
             </inertial>
         </link>
-        <joint name="${prefix}gripper" type="fixed">
-            <origin xyz="0 0 1" rpy="0 0 0"/>
+        <joint name="${prefix}gripper_wrist_fixture" type="fixed">
+            <parent link="${prefix}wrist_link"/>
+            <child link="${prefix}gripper_link"/>
+            <origin xyz="0 0 ${height3 - width}" rpy="0 0 0"/>
+        </joint>
+        <!-- Gripper Link -->
+        <link name="${prefix}gripper_link">
+            <collision>
+                <origin xyz="0 0 ${gripper_thickness/2}" rpy="0 0 0"/>
+                <geometry>
+                    <box size="${gripper_width} ${gripper_breadth} ${gripper_thickness}"/>
+                </geometry>
+            </collision>
+            <visual>
+                <origin xyz="0 0 ${gripper_thickness/2}" rpy="0 0 0"/>
+                <geometry>
+                    <box size="${gripper_width} ${gripper_breadth} ${gripper_thickness}"/>
+                </geometry>
+                <material name="orange"/>
+            </visual>
+            <inertial>
+                <origin xyz="0 0 ${gripper_thickness/2}" rpy="0 0 0"/>
+                <mass value="${mass}"/>
+                <inertia
+                        ixx="${mass / 12.0 * (gripper_width*gripper_breadth + gripper_thickness*gripper_thickness)}" ixy="0.0" ixz="0.0"
+                        iyy="${mass / 12.0 * (gripper_thickness*gripper_thickness + gripper_width*gripper_breadth)}" iyz="0.0"
+                        izz="${mass / 12.0 * (gripper_width*gripper_breadth + gripper_width*gripper_breadth)}"/>
+            </inertial>
+        </link>
+        <joint name="${prefix}gripper" type="prismatic">
+            <origin xyz="${-gripper_width/2 - width/2} 0 ${gripper_thickness}" rpy="0 0 0"/>
             <parent link="${prefix}gripper_link"/>
-            <child link="${prefix}tool_link"/>
-        </joint>
-        <!-- Tool Link -->
-        <link name="${prefix}tool_link">
+            <child link="${prefix}finger_left_link"/>
+            <axis xyz="1 0 0"/>
+            <dynamics damping="0.7"/>
+            <limit lower="0" upper="${gripper_width/2 - finger_thickness}" effort="100" velocity="1.0"/>
+        </joint>
+        <joint name="${prefix}gripper_mimic" type="prismatic">
+            <origin xyz="${-gripper_width/2 - width/2} 0 ${gripper_thickness}" rpy="0 0 0"/>
+            <parent link="${prefix}gripper_link"/>
+            <child link="${prefix}finger_right_link"/>
+            <mimic joint="${prefix}gripper" multiplier="-1" offset="0.5"/>
+            <axis xyz="1 0 0"/>
+            <dynamics damping="0.7"/>
+            <limit lower="${-gripper_width/2 + finger_thickness}" upper="0" effort="100" velocity="1.0"/>
+        </joint>
+        <!-- Finger Links -->
+        <link name="${prefix}finger_left_link">
+            <collision>
+                <origin xyz="${finger_thickness*1.5} 0 ${finger_length/2}" rpy="0 0 0"/>
+                <geometry>
+                    <box size="${finger_thickness} ${gripper_breadth} ${finger_length}"/>
+                </geometry>
+            </collision>
+            <visual>
+                <origin xyz="${finger_thickness*1.5} 0 ${finger_length/2}" rpy="0 0 0"/>
+                <geometry>
+                    <box size="${finger_thickness} ${gripper_breadth} ${finger_length}"/>
+                </geometry>
+                <material name="orange"/>
+            </visual>
+            <inertial>
+                <origin xyz="${finger_thickness*1.5} 0 ${finger_length/2}" rpy="0 0 0"/>
+                <mass value="${mass}"/>
+                <inertia
+                        ixx="${mass / 12.0 * (finger_thickness*gripper_breadth + finger_length*finger_length)}" ixy="0.0" ixz="0.0"
+                        iyy="${mass / 12.0 * (finger_length*finger_length + finger_thickness*gripper_breadth)}" iyz="0.0"
+                        izz="${mass / 12.0 * (finger_thickness*gripper_breadth + finger_thickness*gripper_breadth)}"/>
+            </inertial>
+        </link>
+        <link name="${prefix}finger_right_link">
+            <collision>
+                <origin xyz="${-finger_thickness*1.5} 0 ${finger_length/2}" rpy="0 0 0"/>
+                <geometry>
+                    <box size="${finger_thickness} ${width} ${finger_length}"/>
+                </geometry>
+            </collision>
+            <visual>
+                <origin xyz="${-finger_thickness*1.5} 0 ${finger_length/2}" rpy="0 0 0"/>
+                <geometry>
+                    <box size="${finger_thickness} ${width} ${finger_length}"/>
+                </geometry>
+                <material name="orange"/>
+            </visual>
+            <inertial>
+                <origin xyz="${-finger_thickness*1.5} 0 ${finger_length/2}" rpy="0 0 0"/>
+                <mass value="${mass}"/>
+                <inertia
+                        ixx="${mass / 12.0 * (finger_thickness*width + finger_length*finger_length)}" ixy="0.0" ixz="0.0"
+                        iyy="${mass / 12.0 * (finger_length*finger_length + finger_thickness*width)}" iyz="0.0"
+                        izz="${mass / 12.0 * (finger_thickness*width + finger_thickness*width)}"/>
+            </inertial>
         </link>
     </xacro:macro>
