Commit message: Required for launch, will be transferred to config repo later.

File: hardware/include/ros2_control_demo_description/project_perry/urdf/project_perry_description.urdf.xacro (robot description, xacro)
@@ -14,4 +14,10 @@
   <xacro:property name="caster_wheel_radius" value="0.015" />
   <xacro:property name="z_offset" value="-${base_height/2}" /> <!-- Space btw top of beam and the each joint -->
+  <link name="base_footprint"/>
+  <joint name="base_joint" type="fixed">
+    <parent link="base_footprint"/>
+    <child link="base_link"/>
+    <origin xyz="0 0 0" rpy="0 0 0"/>
+  </joint>
   <!-- Base Link -->
   <link name="${prefix}base_link">
