Commit message: Changed Project Perry xacro's joints to match real model

File: bringup/config/prairie_pioneer.ros2_control.xacro (robot description, xacro)
@@ -10,4 +10,5 @@
           <param name="baud_rate">57600</param>
           <param name="controller_type">ARDUINO</param>
+          <param name="default_speed">1.0</param>
         </hardware>
       </xacro:unless>

File: bringup/config/project_perry.ros2_control.xacro (robot description, xacro)
@@ -20,5 +20,5 @@
         </hardware>
       </xacro:if>
-      <joint name="${prefix}base_yaw_joint">
+      <joint name="base_yaw">
         <command_interface name="velocity"/>
         <command_interface name="position"/>
@@ -28,5 +28,5 @@
         <param name="reduction_factor">13</param>
       </joint>
-      <joint name="${prefix}base_pitch_joint">
+      <joint name="base_pitch">
         <command_interface name="velocity"/>
         <command_interface name="position"/>
@@ -36,5 +36,5 @@
         <param name="reduction_factor">252</param>
       </joint>
-      <joint name="${prefix}elbow_0_joint">
+      <joint name="elbow_pitch">
         <command_interface name="velocity"/>
         <command_interface name="position"/>
@@ -44,9 +44,25 @@
         <param name="reduction_factor">252</param>
       </joint>
-      <gpio name="${prefix}gripper">
+      <joint name="wrist_pitch">
+        <command_interface name="velocity"/>
         <command_interface name="position"/>
         <state_interface name="position"/>
         <state_interface name="velocity"/>
-      </gpio>
+        <param name="motor_id">4</param>
+        <param name="reduction_factor">12</param>
+      </joint>
+      <joint name="wrist_roll">
+        <command_interface name="velocity"/>
+        <command_interface name="position"/>
+        <state_interface name="position"/>
+        <state_interface name="velocity"/>
+        <param name="motor_id">5</param>
+        <param name="reduction_factor">12</param>
+      </joint>
+<!--      <gpio name="${prefix}gripper">-->
+<!--        <command_interface name="position"/>-->
+<!--        <state_interface name="position"/>-->
+<!--        <state_interface name="velocity"/>-->
+<!--      </gpio>-->
     </ros2_control>
   </xacro:macro>
