Commit message: Add bringup materials for can_ppm_controller
NOTE

Currently the controller_manager refuses to operate since it cannot
find the umrt-arm-ros-firmware/ServoControlSystem node. It seems like
it could be an issue in package resolution or an issue in exporting the node
properly so the controller manager can find it.

A few issues we have to get passed to get this working
- Using Generics to select between servo0...7 classes when publishing to
  the babbler.
- Reading the new parameter definitions in <hardware> tags in xacros I added
- Changing the topic prefixes

I recommend the topic structure

    /ppm/<name>/command

where `/ppm` can be replaced with anything the user likes.
Although this will have to be beholden to ros2_control.

File: bringup/config/project_perry.ros2_control.xacro (robot description, xacro)
@@ -2,4 +2,24 @@
 <robot xmlns:xacro="http://www.ros.org/wiki/xacro">
   <xacro:macro name="project_perry_ros2_control" params="name prefix use_mock_hardware">
+    <ros2_control name="${name}-can-ppm" type="system">
+      <hardware>
+        <plugin>umrt-arm-ros-firmware/ServoControlSystem</plugin>
+        <param name="global_subscription_prefix">/arm/ppm</param>
+        <param name="babbler_prefix">/arm/babbler</param>
+        <param name="ppm_gateway_id">0</param>
+      </hardware>
+      <joint name="gripper_servo">
+        <command_interface name="position"/>
+        <state_interface name="position"/>
+        <param name="id">0</param>
+        <param name="initial_position">0.5</param>
+      </joint>
+      <joint name="gripper_solenoid">
+        <command_interface name="position"/>
+        <state_interface name="position"/>
+        <param name="id">1</param>
+        <param name="initial_position">0.5</param>
+      </joint>
+    </ros2_control>
     <ros2_control name="${name}" type="system">
       <xacro:unless value="${use_mock_hardware}">
